File: circuit.sch (EAGLE design)
At the start: 3 parts, among them IC1 7805T, U1 MCP4725

Commit message: Working on the schematic.
Parts:
- removed CPU: ARDUINO_PRO_MINI, SparkFun-Boards:ARDUINO_PRO_MINI
- removed IC1: 7805T, adafruit:7805T
- added B1: ARDUINO_PRO_MINI, SparkFun-Boards:ARDUINO_PRO_MINI
- added C1: 10uF, microbuilder:CAP_CERAMIC_0805MP
- added IC2: 7805DT, adafruit:7805DT
- added JP1: (no value), jumper:JP4E
- added R1, R2, R3: 4.7k, adafruit:R-US_M1206
- added R4: 10k, adafruit:R-US_M1206
- added U2: MB85RC256VPF-G-JNERE2, microbuilder:FRAM_SOIC8_I2C
Connections:
- new net ETH: B1.*5, JP1.3, R1.1
- new net OUT: JP1.4, U1.VOUT
- new net VIN: IC2.VI, JP1.1
- net GND: now also B1.GND@2, C1.2, IC2.GND, JP1.2, R4.1, U1.VSS, U2.GND; no longer CPU.GND@2, IC1.GND
- net N$1: now also B1.A5, R2.1, U2.SCL; no longer CPU.A4
- net N$2: now also B1.A4, R3.1, U2.SDA; no longer CPU.A5
- net N$4: now also R4.2, U1.AO; no longer CPU.VCC, IC1.VO
- net VCC: now also B1.VCC, C1.1, IC2.VO, R1.2, R2.2, R3.2, U1.VDD, U2.VCC; no longer IC1.VI
Other:
- moved on the sheet: U1
